File: tinyg_g2_breakout_v1.brd (EAGLE design)
At the start: 83.8 x 52.8 mm, 27 parts

Commit message: latest changes
Parts:
- removed C10: 0.1uf, SparkFun-Passives:CAP-PTH-SMALL
- removed R10: 10k, SparkFun-Passives:AXIAL-0.3
- J2: device SparkFun-Connectors:1X04 -> SparkFun-Connectors:1X03
- J3: device SparkFun-Connectors:1X04 -> SparkFun-Connectors:1X05
- moved J3 2.60 mm to (68.3, 20.4)
- moved U$2 1.77 mm to (10.3, 16.9)
- moved U$1 1.41 mm to (20.0, 18.8)
- moved J2 0.10 mm to (68.3, 11.9)
Connections:
- net 3.3V: no longer R10.P$2
- net COOLON: now also J3.1; no longer C7.2, J2.1, R7.P$1
- net GBLCYST: now also C7.2, J2.1, R7.P$1; no longer C8.2, J2.2, R8.P$1
- net GBLENAB: now also J3.5; no longer J3.4
- net GBLFRH: now also C8.2, J2.2, R8.P$1; no longer C9.2, J2.3, R9.P$1
- net GBLRST: now also C9.2, J2.3, R9.P$1; no longer C10.2, J2.4, R10.P$1
- net GND: no longer C10.1
- net SPENAB: now also J3.3; no longer J3.2
- net SPNDIR: now also J3.2; no longer J3.1
- net SPPWM: now also J3.4; no longer J3.3
Routing:
- net XMN: track 51.9 -> 68.0 mm
- net SPNDIR: track 68.0 -> 83.6 mm
- net SPENAB: track 64.4 -> 79.3 mm
- net SPPWM: track 60.8 -> 74.2 mm
- net YMX: track 34.5 -> 47.4 mm
- net COOLON: track 49.0 -> 41.0 mm
- net YMN: track 50.2 -> 44.2 mm
- net GBLRST: track 49.3 -> 45.6 mm
- net GBLCYST: track 42.8 -> 46.1 mm
- net GBLENAB: track 60.5 -> 63.3 mm
- net 3.3V: track 61.5 -> 59.5 mm
- net ZMX: track 29.0 -> 30.7 mm
- net ZMN: track 28.6 -> 30.1 mm
- net GBLFRH: track 44.4 -> 43.3 mm
Other:
- board text added: "0"
- board text added: "1"
- board text added: "10"
- board text added: "11"
- board text added: "12"
- board text added: "13"
- board text added: "14"
- board text added: "15"
- board text added: "16"
- board text added: "17"
- board text added: "18"
- board text added: "19"
- board text added: "2"
- board text added: "20"
- board text added: "21"
- board text added: "22"
- board text added: "3"
- board text added: "3.3V"
- board text added: "31"
- board text added: "33"
- board text added: "35"
- board text added: "37"
- board text added: "39"
- board text added: "4"
- board text added: "41"
- board text added: "43"
- board text added: "45"
- board text added: "47"
- board text added: "49"
- board text added: "5"
- board text added: "51"
- board text added: "52"
- board text added: "53"
- board text added: "5V"
- board text added: "6"
- board text added: "7"
- board text added: "8"
- board text added: "9"
- board text added: "A0"
- board text added: "A1"
- board text added: "A10"
- board text added: "A11"
- board text added: "A2"
- board text added: "A3"
- board text added: "A4"
- board text added: "A5"
- board text added: "A6"
- board text added: "A7"
- board text added: "A8"
- board text added: "A9"
- board text added: "AREF"
- board text added: "IOREF"
- board text added: "RESET"
- board text added: "SCL1"
- board text added: "SDA1"
- board text added: "Vin"
