File: tinyg_g2_breakout_v1.sch (EAGLE design)
At the start: 25 parts

Commit message: latest changes
Parts:
- removed C10: 0.1uf, SparkFun-Passives:CAPPTH
- removed R10: 10k, SparkFun-Passives:RESISTORAXIAL-0.3
- J2: device SparkFun-Connectors:M04PTH -> SparkFun-Connectors:M03PTH
- J3: device SparkFun-Connectors:M04PTH -> SparkFun-Connectors:M05PTH
Connections:
- net 3.3V: no longer R10.2
- net COOLON: now also J3.1; no longer C7.2, J2.1, R7.1
- net GBLCYST: now also C7.2, J2.1, R7.1; no longer C8.2, J2.2, R8.1
- net GBLENAB: now also J3.5; no longer J3.4
- net GBLFRH: now also C8.2, J2.2, R8.1; no longer C9.2, J2.3, R9.1
- net GBLRST: now also C9.2, J2.3, R9.1; no longer C10.2, J2.4, R10.1
- net GND: no longer C10.1
- net SPENAB: now also J3.3; no longer J3.2
- net SPNDIR: now also J3.2; no longer J3.1
- net SPPWM: now also J3.4; no longer J3.3
