File: tinyg_g2_breakout.brd (EAGLE design)
At the start: 83.8 x 52.8 mm, 25 parts

Commit message: Updated files
Parts:
- added FRAME1: v1, SparkFun-Aesthetics:CREATIVE_COMMONS
- moved J4 5.04 mm to (63.3, 5.78)
- moved J1 5.00 mm to (63.3, 46.9)
- moved J2 5.00 mm to (63.3, 11.9)
- moved J3 5.00 mm to (63.3, 20.4)
- moved C5 3.00 mm to (38.0, 42.0)
- moved C6 3.00 mm to (38.0, 45.0)
Routing:
- net YMX: track 47.4 -> 30.3 mm
- net SPNDIR: track 83.6 -> 67.8 mm
- net SPENAB: track 79.3 -> 64.5 mm
- net XMN: track 68.0 -> 54.9 mm
- net XMX: track 53.4 -> 40.4 mm
- net SPPWM: track 74.2 -> 62.1 mm
- net 3.3V: track 59.5 -> 71.4 mm
- net ZMX: track 30.7 -> 19.8 mm
- net GBLCYST: track 46.1 -> 36.5 mm
- net COOLON: track 41.0 -> 32.6 mm
- net YMN: track 44.2 -> 36.1 mm
- net GBLRST: track 45.6 -> 39.9 mm
- net GBLENAB: track 63.3 -> 58.0 mm
- net ZMN: track 30.1 -> 26.7 mm
Other:
- board size 83.8 x 52.8 mm -> 84.8 x 52.8 mm
- board text added: "mike@machadolab.com"
- board text added: "v2"
- board text removed: "A10"
- board text removed: "A11"
- board text removed: "v1"
